Commit message: 20231204

File: my_lite6_description/urdf/lite6_robot.urdf.xacro (robot description, xacro)
@@ -1,6 +1,10 @@
 <?xml version="1.0"?>
 <robot xmlns:xacro="http://wiki.ros.org/xacro" name="lite6_robot">
+  <!--
   <xacro:arg name="prefix" default="arm_"/>
   <xacro:arg name="hw_ns" default="xarm"/>
+  -->
+  <xacro:arg name="prefix" default=""/>
+  <xacro:arg name="hw_ns" default=""/>
   <xacro:arg name="limited" default="false"/>
   <xacro:arg name="effort_control" default="false"/>
@@ -108,5 +112,5 @@
   <link name="tcp_link" />
   <joint name="tool_link" type="fixed">
-    <parent link="arm_link_eef" />
+    <parent link="link_eef" />
     <child link="tcp_link" />
     <origin xyz="0.0 0.0 0.0" rpy="0.0 ${-pi/2} 0.0"/>

Commit message: 20231205

File: my_lite6_description/urdf/lite6_robot.urdf.xacro (robot description, xacro)
@@ -1,4 +1,4 @@
 <?xml version="1.0"?>
-<robot xmlns:xacro="http://wiki.ros.org/xacro" name="lite6">
+<robot xmlns:xacro="http://wiki.ros.org/xacro" name="lite6_robot">
   <!--
   <xacro:arg name="prefix" default="arm_"/>
@@ -99,12 +99,30 @@
   </link>
   <joint name="baseplate_joint" type="fixed">
-    <origin xyz="0 0 0" />
+    <origin xyz="0 0 -0.015" />
     <parent link="world" />
     <child link="baseplate_link" />
   </joint>
+  <link name="mountingplate_link">
+    <visual>
+      <origin xyz="0 0 0.0" />
+      <geometry>
+        <box size="0.130 0.190 0.005" />
+      </geometry>
+      <material name="red"/>
+    </visual>
+    <inertial>
+      <mass value="1"/>
+      <xacro:box_inertia m="1" x="0.130" y="0.190" z="0.005"/>
+    </inertial>
+  </link>
+  <joint name="mountingplate_joint" type="fixed">
+    <origin xyz="-0.285 0.0 0.0175" />
+    <parent link="baseplate_link" />
+    <child link="mountingplate_link" />
+  </joint>
   <link name="xarm_link"/>
   <joint name="base_plate_to_xarm_joint" type="fixed">
-    <origin xyz="-0.2 0.0 0.021" />
-    <parent link="baseplate_link" />
+    <origin xyz="-0.0 0.0 0.0025" />
+    <parent link="mountingplate_link" />
     <child link="xarm_link" />
   </joint>

Commit message: 20231206

File: my_lite6_description/urdf/lite6_robot.urdf.xacro (robot description, xacro)
@@ -132,5 +132,5 @@
     <parent link="link_eef" />
     <child link="tcp_link" />
-    <origin xyz="0.0 0.0 0.0" rpy="0.0 ${-pi/2} 0.0"/>
+    <origin xyz="0.0 0.0 0.0" rpy="0.0 0.0 0.0"/>
   </joint>
 </robot>

Commit message: 20240412

File: my_lite6_description/urdf/lite6_robot.urdf.xacro (robot description, xacro)
@@ -97,4 +97,9 @@
       <xacro:box_inertia m="10" x="1.1" y="0.7" z="0.03"/>
     </inertial>
+    <collision>
+      <geometry>
+        <box size="0.7 1.1 0.03" />
+      </geometry>
+    </collision>
   </link>
   <joint name="baseplate_joint" type="fixed">
@@ -115,4 +120,9 @@
       <xacro:box_inertia m="1" x="0.130" y="0.190" z="0.005"/>
     </inertial>
+    <collision>
+      <geometry>
+        <box size="0.13 0.19 0.005" />
+      </geometry>
+    </collision>
   </link>
   <joint name="mountingplate_joint" type="fixed">
